File: plank.kicad_pcb (KiCad board)
At the start: 2 copper layers, 148.6 x 24.1 mm, 108 parts, among them P1 3.3V, P10 SW4, P11 LED1, P12 ANA1, P13 ANA5, P14 SW5, P15 LED2, P16 ANA2, P17 ANA6, P18 SW6, P19 LED3, P2 I2C, P20 SW7, P21 LED4, P22 ANA3, P23 ANA7, P24 LED5, P25 LED6, P26 LED7, P3 SW0, P4 SW1, P5 SW2, P6 SW3, P7 LED0, P8 ANA0, P9 ANA4, Q1 Q_PNP_BCE, U1 MAX7313, U2 ADS1015, U3 ADS1015, U4 24C16

Commit message: Taped out 20 cards
Parts:
- removed C3: C, Capacitors_SMD:C_0603
- removed R24: 10k, Resistors_SMD:R_0603
- removed U3: ADS1015, Housings_SSOP:MSOP-10_3x3mm_Pitch0.5mm
- removed U4: 24C16, SMD_Packages:SOIC-8-N
- added P27: CONN_01X05, Pin_Headers:Pin_Header_Straight_1x05, F.Cu at (143.5, 86.4)
- added R33: DNM, Resistors_SMD:R_0603, F.Cu at (154.2, 70.6)
- added R34: DNM, Resistors_SMD:R_0603, F.Cu at (152.1, 70.6)
- F1: footprint Capacitors_SMD:C_0603_HandSoldering -> Capacitors_SMD:C_1206_HandSoldering
- Q1: value Q_PNP_BCE -> Q_PNP_BEC
- U2: value ADS1015 -> MCP3008; footprint Housings_SSOP:MSOP-10_3x3mm_Pitch0.5mm -> Housings_SOIC:SOIC-16_3.9x9.9mm_Pitch1.27mm
- moved C2 15.9 mm to (156.5, 75.9), turned to 270 degrees
- moved U2 8.68 mm to (151.6, 79.2)
- moved C4 7.86 mm to (156.2, 82.6), turned to 270 degrees
- moved F1 4.96 mm to (165.1, 78.7), turned to 90 degrees
- moved Q1 0.28 mm to (161.5, 78.2)
Connections:
- C14 pad 1: Net-(C14-Pad1) -> /ana0
- C15 pad 1: Net-(C15-Pad1) -> /ana4
- C16 pad 1: Net-(C16-Pad1) -> /ana1
- C17 pad 1: Net-(C17-Pad1) -> /ana5
- C18 pad 1: Net-(C18-Pad1) -> /ana2
- C19 pad 1: Net-(C19-Pad1) -> /ana6
- C20 pad 1: Net-(C20-Pad1) -> /ana3
- C21 pad 1: Net-(C21-Pad1) -> /ana7
- Q1 pad 2: Net-(D3-Pad2) -> Net-(F1-Pad1)
- Q1 pad 3: Net-(F1-Pad1) -> Net-(D3-Pad2)
- R16 pad 1: Net-(C16-Pad1) -> /ana1
- R17 pad 1: Net-(C20-Pad1) -> /ana3
- R18 pad 1: Net-(C17-Pad1) -> /ana5
- R19 pad 1: Net-(C21-Pad1) -> /ana7
- R20 pad 1: Net-(C14-Pad1) -> /ana0
- R21 pad 1: Net-(C18-Pad1) -> /ana2
- R22 pad 1: Net-(C15-Pad1) -> /ana4
- R23 pad 1: Net-(C19-Pad1) -> /ana6
- U2 pad 1: GND -> /ana0
- U2 pad 10: /scl -> /~CS
- U2 pad 2: (no net) -> /ana1
- U2 pad 3: GND -> /ana2
- U2 pad 4: Net-(C14-Pad1) -> /ana3
- U2 pad 5: Net-(C16-Pad1) -> /ana4
- U2 pad 6: Net-(C18-Pad1) -> /ana5
- U2 pad 7: Net-(C20-Pad1) -> /ana6
- U2 pad 8: +3V3 -> /ana7
- U2 pad 9: /sda -> GND
Routing:
- net /ana0: track 0.00 -> 131.9 mm, vias 0 -> 2
- net Net-(C14-Pad1): track 119.9 -> 0.00 mm, vias 2 -> 0
- net /ana1: track 0.00 -> 113.3 mm, vias 0 -> 2
- net Net-(C16-Pad1): track 104.0 -> 0.00 mm, vias 2 -> 0
- net GND: track 980.3 -> 1083.3 mm, vias 67 -> 73
- net Net-(C18-Pad1): track 97.7 -> 0.00 mm, vias 2 -> 0
- net /ana2: track 0.00 -> 97.0 mm, vias 0 -> 2
- net /ana3: track 0.00 -> 80.7 mm, vias 0 -> 2
- net Net-(C20-Pad1): track 79.7 -> 0.00 mm, vias 2 -> 0
- net Net-(C15-Pad1): track 65.4 -> 0.00 mm, vias 2 -> 0
- net /ana4: track 0.00 -> 65.0 mm, vias 0 -> 2
- net Net-(C17-Pad1): track 49.6 -> 0.00 mm, vias 2 -> 0
- net (no net): track 49.5 -> 0.00 mm
- net /ana5: track 0.00 -> 48.9 mm, vias 0 -> 2
- net Net-(C19-Pad1): track 39.8 -> 0.00 mm, vias 2 -> 0
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Other:
- board text added: "CLK"
- board text added: "COSMO plank 1.0 3.3 V supply and I/O LED's from 3.3V to round pad LED max 50 mA Buttons from GND to square pad"
- board text added: "MISO"
- board text added: "MOSI"
- board text added: "~CS"
- board text removed: "COSMO plank 1.0 3.3 V supply and I/O LED's from 3.3V to round pad LED max 55 mA Buttons from GND to square pad"

Commit message: New version of the plank
Routing:
- net GND: track 1083.3 -> 1224.0 mm, vias 73 -> 85
- net +3V3: track 577.3 -> 578.1 mm
Other:
- board text added: "B+"
- board text added: "COSMO plank 1.1"
- board text added: "COSMO plank 1.1 3.3 V supply and I/O LED's from 3.3V to round pad LED max 50 mA Buttons from GND to square pad"
- board text added: "L-"
- board text removed: "COSMO plank 1.0"
- board text removed: "COSMO plank 1.0 3.3 V supply and I/O LED's from 3.3V to round pad LED max 50 mA Buttons from GND to square pad"
