File: plank.sch (KiCad schematic (older format))
At the start: 108 parts, among them P1 3.3V, P10 SW4, P11 LED1, P12 ANA1, P13 ANA5, P14 SW5, P15 LED2, P16 ANA2, P17 ANA6, P18 SW6, P19 LED3, P2 I2C, P20 SW7, P21 LED4, P22 ANA3, P23 ANA7, P24 LED5, P25 LED6, P26 LED7, P3 SW0, P4 SW1, P5 SW2, P6 SW3, P7 LED0, P8 ANA0, P9 ANA4, Q1 Q_PNP_BCE, U1 MAX7313, U2 ADS1015, U3 ADS1015, U4 24C16

Commit message: Taped out 20 cards
Parts:
- removed C3: C, Capacitors_SMD:C_0603, symbol C
- removed Q1: Q_PNP_BCE, TO_SOT_Packages_SMD:SOT-23, symbol Q_PNP_BCE
- removed R24: 10k, Resistors_SMD:R_0603, symbol R
- removed U2, U3: ADS1015, Housings_SSOP:MSOP-10_3x3mm_Pitch0.5mm, symbol ADS1015-RESCUE-plank
- removed U4: 24C16, SMD_Packages:SOIC-8-N, symbol 24C16
- added P27: CONN_01X05, Pin_Headers:Pin_Header_Straight_1x05, symbol CONN_01X05
- added Q?: Q_PNP_BEC, symbol Q_PNP_BEC
- added R33, R34: DNM, Resistors_SMD:R_0603, symbol R
- added U2: MCP3008, Housings_SOIC:SOIC-16_3.9x9.9mm_Pitch1.27mm, symbol MCP3008
- F1: footprint Capacitors_SMD:C_0603_HandSoldering -> Capacitors_SMD:C_1206_HandSoldering
Connections:
- net +3V3: now also R33.2, R34.2, U2.15 (VREF), U2.16 (VDD)
- net GND: now also P27.1 (P1), U2.14 (AGND), U2.9 (DGND)
- net scl: now also R33.1
- net sda: now also R34.1
- net at F1.1, P1.2 (P2): now also Q?.2 (E)
- net at R2.2: now also Q?.1 (B)
- net at D3.2 (A): now also Q?.3 (C)
- net ana0: now reaches C14.1, R20.1
- net ana0: now also U2.1 (CH0)
- net ana1: now reaches C16.1, R16.1
- net ana1: now also U2.2 (CH1)
- net ana2: now reaches C18.1, R21.1
- net ana2: now also U2.3 (CH2)
- net ana3: now reaches C20.1, R17.1
- net ana3: now also U2.4 (CH3)
- net ana4: now reaches C15.1, R22.1
- net ana4: now also U2.5 (CH4)
- net ana5: now reaches C17.1, R18.1
- net ana5: now also U2.6 (CH5)
- net ana6: now reaches C19.1, R23.1
- net ana6: now also U2.7 (CH6)
- net ana7: now reaches C21.1, R19.1
- net ana7: now also U2.8 (CH7)
- new net MISO: P27.3 (P3), U2.12 (DOUT)
- new net MOSI: P27.4 (P4), U2.11 (DIN)
- new net spiclk: P27.2 (P2), U2.13 (CLK)
- new net ~CS: P27.5 (P5), U2.10 (~CS~/SHDN)
- no-connect marks 2 -> 0
Other:
- note removed: "addr: 1001000"
- note removed: "addr: 1001001"
- note removed: "addr: 1010000"

Commit message: New version of the plank
Parts:
- Q1: renamed from Q?; footprint (none) -> TO_SOT_Packages_SMD:SOT-23
Changed lines of the file:
@@
 Connection ~ 2350 4050
 $Comp
-L Q_PNP_BEC Q?
+L Q_PNP_BEC Q1
 U 1 1 580DE8E0
 P 1600 800
-F 0 "Q?" H 1900 850 50  0000 R CNN
+F 0 "Q1" H 1900 850 50  0000 R CNN
 F 1 "Q_PNP_BEC" H 2200 750 50  0000 R CNN
-F 2 "" H 1800 900 50  0000 C CNN
+F 2 "TO_SOT_Packages_SMD:SOT-23" H 1800 900 50  0001 C CNN
 F 3 "" H 1600 800 50  0000 C CNN
 	1    1600 800
